File: hw/vco1/vco1.kicad_sch (KiCad schematic)
At the start: 81 parts, among them J1 Conn_02x08_Odd_Even, Q1 DNP, SW1 SW_SPDT, U1 SSI2131, U2 TL431BCDBZR, U4 TL072HxD, U5 TL072HxD

Commit message: As built, fixed a couple of issues
Parts:
- removed R8: 1k, Resistor_SMD:R_0603_1608Metric_Pad0.98x0.95mm_HandSolder, symbol Device:R
- added C16: 100n, Capacitor_SMD:C_0805_2012Metric_Pad1.18x1.45mm_HandSolder, symbol Device:C
- added R34, R35: 10k, Resistor_SMD:R_0603_1608Metric_Pad0.98x0.95mm_HandSolder, symbol Device:R
- added R36: 150k, Resistor_SMD:R_0603_1608Metric_Pad0.98x0.95mm_HandSolder, symbol Device:R
- C1, Q1, R23, R24: now not fitted
- C7: value 2.2u -> 100n
- R29: value 0 -> 49k9
- R32, R33: value 20k -> 39k
Connections:
- net +12V: now also R36.2
- net +2V5: now also R35.1; no longer R32.1
- net EXPO_FREQ: now also R36.1
- net at R4.1, U4.7: now also C16.1
- net at J_PULSE1.T: now also C16.2
- net 1.25V renamed OPREF
- new net: R34.2, R35.2
- new net: R32.1, R34.1
Other:
- note added: "0.995V, matching the opamp gain resistors"
- note added: "100n gives 0.7-25 Hz range, stability unimportant"
- note added: "80µA bias to set base to 27 Hz"
- note added: "FIXME: connect to other side of R7"
- note added: "Nominally 24.3k"
- note added: "no cap! makes unstable"
- note removed: "LFO range with uF stability unimportant"
- moved on the sheet: R32
