File: hw/bananabus/bananabus.kicad_pcb (KiCad board)
At the start: 2 copper layers, 95 x 46 mm, 19 parts, among them J1 Conn_02x08_Odd_Even, J2 Conn_02x08_Odd_Even, J3 Conn_02x08_Odd_Even, J4 Conn_02x08_Odd_Even, J5 Conn_01x01_Socket, J6 Conn_01x01_Socket, J7 Conn_01x01_Socket, J8 Conn_01x01_Socket

Commit message: Banana bus gerbers
Routing:
- net GND: track 831.5 -> 18.1 mm, vias 0 -> 1
- net +5V: track 256.4 -> 266.0 mm
- net +12V: track 81.5 -> 90.5 mm
- net -12V: track 288.4 -> 294.9 mm
- net Net-(D3-K): track 0.00 -> 4.05 mm
- net Net-(D2-K): track 0.00 -> 4.05 mm
- net Net-(D1-K): track 0.00 -> 4.05 mm
