File: hw/develboard_12hp/develboard_12hp.kicad_pcb (KiCad board)
At the start: 2 copper layers, 60 x 110 mm, 59 parts, among them J1 Conn_02x08_Odd_Even, U4 TL072HxD, U5 TL072HxD

Commit message: Stupid hurried development board
Parts:
- removed C2, C3: 10u, Capacitor_THT:CP_Radial_D5.0mm_P2.50mm
- removed H1, H2, H3: MountingHole, Holes:MountingHole_3.2mm_M3_Pad
- removed JP1: jumper, Jumper:SolderJumper-2_P1.3mm_Bridged2Bar_Pad1.0x1.5mm
- added C5: 0, Capacitor_SMD:C_0603_1608Metric_Pad1.08x0.95mm_HandSolder, B.Cu at (136.5, 121.1)
- added C6: 0, Capacitor_SMD:C_0603_1608Metric_Pad1.08x0.95mm_HandSolder, B.Cu at (126.7, 121.3)
- added C7: 0, Capacitor_SMD:C_0603_1608Metric_Pad1.08x0.95mm_HandSolder, B.Cu at (93.4, 121.2)
- added C8: 0, Capacitor_SMD:C_0603_1608Metric_Pad1.08x0.95mm_HandSolder, B.Cu at (83.2, 121.1)
- added G***: LOGO, elemental:elemental-4mm, F.Cu at (82.5, 128.0)
- added J2: Conn_01x04, Connector_PinHeader_2.54mm:PinHeader_1x04_P2.54mm_Vertical, B.Cu at (102.3, 116.5)
- added J3: Conn_01x04, Connector_PinHeader_2.54mm:PinHeader_1x04_P2.54mm_Vertical, B.Cu at (112.5, 116.5)
- added J4: Conn_01x04, Connector_PinHeader_2.54mm:PinHeader_1x04_P2.54mm_Vertical, B.Cu at (110.0, 50.1)
- added J5: Conn_01x04, Connector_PinHeader_2.54mm:PinHeader_1x04_P2.54mm_Vertical, B.Cu at (92.2, 116.5)
- added J6: Conn_01x04, Connector_PinHeader_2.54mm:PinHeader_1x04_P2.54mm_Vertical, B.Cu at (82.0, 116.5)
- added J7: Conn_01x04, Connector_PinHeader_2.54mm:PinHeader_1x04_P2.54mm_Vertical, B.Cu at (130.3, 116.5)
- added TP1: TestPoint, Holes:TP_0.9mm, F.Cu at (94.1, 50.5)
- J_CV3: renamed from J_IN3; moved to F.Cu
- J_CV4: renamed from J_IN4; moved to F.Cu
- J_IN2: renamed from J_TRI2; moved to F.Cu
- RV3, RV4: moved to F.Cu
- moved J_CV4 120.2 mm to (130.0, 132.0)
- moved R21 120.0 mm to (133.2, 128.6), turned to -90 degrees
- moved R30 119.7 mm to (134.5, 120.9), turned to 90 degrees
- moved R29 118.8 mm to (132.6, 121.3), turned to 90 degrees
- moved R8 115.6 mm to (131.0, 136.8), turned to -90 degrees
- moved J_IN2 113.8 mm to (95.0, 148.0)
- moved R28 111.9 mm to (124.2, 121.4), turned to 90 degrees
- moved R20 111.7 mm to (122.8, 128.3), turned to -90 degrees
- moved R27 110.9 mm to (122.2, 121.4), turned to 90 degrees
- moved R16 110.3 mm to (135.7, 49.6), turned to 90 degrees
- moved R17 106.8 mm to (131.4, 49.7), turned to -90 degrees
- moved J_CV3 104.1 mm to (120.0, 132.0)
- moved RV4 103.7 mm to (133.0, 46.0), turned to 90 degrees
- moved C1 99.4 mm to (117.4, 128.0), turned to -90 degrees
- moved C4 95.8 mm to (117.3, 121.1), turned to -90 degrees
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- renumbered J_IN1 to J_CV1, J_IN2 to J_CV2, J_TRI1 to J_IN1
Connections:
- net Net-(R22-Pad1) renamed /CV1
- net Net-(R24-Pad1) renamed /CV2
- net Net-(R27-Pad1) renamed /CV3
- net Net-(R29-Pad1) renamed /CV4
- J1 pad 14: Net-(J1-Pin_14) -> unconnected-(J1-Pin_14-Pad14)
- R23 pad 2: unconnected-(R23-Pad2) -> GND
- R25 pad 2: unconnected-(R25-Pad2) -> GND
- R28 pad 2: unconnected-(R28-Pad2) -> GND
- R30 pad 2: unconnected-(R30-Pad2) -> GND
- RV4 pad 2: /POT3 -> /POT4
- U5 pad 3: unconnected-(U5A-+-Pad3) -> GND
- U5 pad 5: unconnected-(U5B-+-Pad5) -> GND
Routing:
- net (no net): track 0.00 -> 223.5 mm, vias 0 -> 529
- net +5V: track 0.00 -> 119.7 mm
- net -12V: track 0.00 -> 107.0 mm, vias 0 -> 2
- net +3.3V: track 0.00 -> 50.5 mm
- net /CV4: track 0.00 -> 45.2 mm
- net /CV3: track 0.00 -> 35.4 mm, vias 0 -> 1
- net +12V: track 0.00 -> 30.8 mm, vias 0 -> 2
- net /ADC_IN2: track 0.00 -> 29.5 mm
- net /POT4: track 0.00 -> 27.4 mm
- net /POT1: track 0.00 -> 26.5 mm
- net /DAC_OUT1: track 0.00 -> 25.9 mm
- net Net-(J_IN1-PadT): track 0.00 -> 24.9 mm
- net Net-(R4-Pad1): track 0.00 -> 24.6 mm, vias 0 -> 2
- net Net-(R2-Pad1): track 0.00 -> 21.3 mm, vias 0 -> 2
- net /ADC_IN1: track 0.00 -> 18.4 mm
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