File: hw/develboard_12hp/develboard_12hp.kicad_sch (KiCad schematic)
At the start: 59 parts, among them J1 Conn_02x08_Odd_Even, U4 TL072HxD, U5 TL072HxD

Commit message: Stupid hurried development board
Parts:
- removed C2, C3: 10u, Capacitor_THT:CP_Radial_D5.0mm_P2.50mm, symbol Device:C_Polarized
- removed JP1: jumper, Jumper:SolderJumper-2_P1.3mm_Bridged2Bar_Pad1.0x1.5mm, symbol Jumper:SolderJumper_2_Bridged
- added C5, C6, C7, C8: 0, Capacitor_SMD:C_0603_1608Metric_Pad1.08x0.95mm_HandSolder, symbol Device:C
- added J2, J3, J4, J5, J6, J7: Conn_01x04, Connector_PinHeader_2.54mm:PinHeader_1x04_P2.54mm_Vertical, symbol Connector_Generic:Conn_01x04
- added TP1: TestPoint, Holes:TP_0.9mm, symbol Connector:TestPoint
- renumbered J_IN1 to J_CV1, J_IN2 to J_CV2, J_IN3 to J_CV3, J_IN4 to J_CV4, J_TRI1 to J_IN1, J_TRI2 to J_IN2
Connections:
- net +12V: now also J6.3 (Pin_3), J7.3 (Pin_3)
- net +3.3V: now also TP1.1
- net +5V: now also J6.4 (Pin_4), J7.4 (Pin_4)
- net -12V: now also J6.1 (Pin_1), J7.1 (Pin_1)
- net ADC_IN1: now also J2.1 (Pin_1)
- net ADC_IN2: now also J2.3 (Pin_3)
- net DAC_OUT1: now also J3.1 (Pin_1)
- net DAC_OUT2: now also J3.3 (Pin_3)
- net GND: now also R23.2, R25.2, R28.2, R30.2, U5.3 (+), U5.5 (+), C5.2, C6.2, C7.2, C8.2, J2.2 (Pin_2), J2.4 (Pin_4), J3.2 (Pin_2), J3.4 (Pin_4), J6.2 (Pin_2), J7.2 (Pin_2)
- net POT1: now also J4.1 (Pin_1)
- net POT2: now also J4.2 (Pin_2)
- net POT3: now also J4.3 (Pin_3); no longer RV4.2
- net CV4: now reaches R29.1, R30.1
- net CV4: now also C5.1, J5.4 (Pin_4)
- net CV1: now reaches R22.1, R23.1
- net CV1: now also C8.1, J5.1 (Pin_1)
- net CV3: now reaches R27.1, R28.1
- net CV3: now also C6.1, J5.3 (Pin_3)
- net CV2: now reaches R24.1, R25.1
- net CV2: now also C7.1, J5.2 (Pin_2)
- new net POT4: J4.4 (Pin_4), RV4.2
