File: hw/flexmodule1/flexmodule1.kicad_pcb (KiCad board)
At the start: 2 copper layers, 19 x 112 mm, 66 parts, among them J1 AudioJack2, J2 AudioJack2, J3 AudioJack2, J4 AudioJack2, J5 AudioJack2, J6 rack_power, J7 SWD, J8 USB_B_Micro, J9 jack, SW1 mode, SW2 bootloader, U1 STM32G431K6Tx, U2 ADP7142AUJZ-5.0, U4 ADP7142AUJZ-3.3, U6 74HCT541, Y1 Crystal

Commit message: Change to a bigger LDO
Use a bigger 5V regulator with 12V input tolerance, so it might be
able to dissipate more heat. Not sure how warm this is going to get.
Parts:
- removed TP3, TP4, TP5: tp, Holes:TP_0.9mm
- removed U4: ADP7142AUJZ-3.3, Package_TO_SOT_SMD:TSOT-23-5
- added TP1: 5V, Holes:TP_0.9mm, F.Cu at (145.5, 121.1)
- added U3: TLV70233_SOT23-5, Package_TO_SOT_SMD:SOT-23-5, B.Cu at (140.3, 93.0)
- C2: value C -> 10u; footprint Capacitor_SMD:C_0603_1608Metric_Pad1.08x0.95mm_HandSolder -> Capacitor_THT:CP_Radial_D5.0mm_P2.50mm; moved to F.Cu
- C4: value C -> 4.7u; footprint Capacitor_SMD:C_0603_1608Metric_Pad1.08x0.95mm_HandSolder -> Capacitor_SMD:C_1206_3216Metric_Pad1.33x1.80mm_HandSolder
- SW2: footprint Button_Switch_THT:SW_PUSH_6mm -> Button_Switch_SMD:SW_SPST_B3S-1000
- TP2: value tp -> 3V
- U2: value ADP7142AUJZ-5.0 -> TLV1117-50IDCYR; footprint Package_TO_SOT_SMD:TSOT-23-5 -> Package_TO_SOT_SMD:SOT-223-3_TabPin2
- moved TP2 35.9 mm to (148.5, 105.0)
- moved G*** 10.3 mm to (147.2, 79.0)
- moved R8 9.63 mm to (139.8, 97.4), turned to 180 degrees
- moved C4 9.01 mm to (145.0, 94.0), turned to 180 degrees
- moved D2 8.28 mm to (139.0, 100.5), turned to -90 degrees
- moved C2 7.91 mm to (148.0, 91.5), turned to 180 degrees
- moved SW2 7.85 mm to (143.0, 101.0), turned to 180 degrees
- moved D1 5.70 mm to (141.0, 100.5), turned to -90 degrees
- moved U2 5.70 mm to (145.5, 99.5)
- moved C1 0.50 mm to (140.5, 89.5)
- turned C7 to 0 degrees
Connections:
- C2 pad 1: +12V -> /VIN
- D1 pad 1: +12V -> /VIN
- D2 pad 1: +12V -> /VIN
- TP2 pad 1: Net-(U1-PB5) -> +3.3V
- U1 pad 27: Net-(U1-PB4) -> unconnected-(U1-PB4-Pad27)
- U1 pad 28: Net-(U1-PB5) -> unconnected-(U1-PB5-Pad28)
- U1 pad 29: Net-(U1-PB6) -> unconnected-(U1-PB6-Pad29)
- U1 pad 30: Net-(U1-PB7) -> unconnected-(U1-PB7-Pad30)
- U2 pad 1: +12V -> GND
- U2 pad 2: GND -> +5V
- U2 pad 3: unconnected-(U2-EN-Pad3) -> /VIN
Routing:
- net +5V: track 40.1 -> 64.6 mm
- net +3.3V: track 104.1 -> 126.6 mm, vias 5 -> 6
- net /VIN: track 0.00 -> 18.5 mm, vias 0 -> 2
- net +12V: track 17.1 -> 0.00 mm
- net /BOOT0: track 31.5 -> 41.9 mm, vias 1 -> 3
- net /USB_VBUS: track 11.0 -> 4.26 mm
- net /OUT4: track 58.1 -> 54.1 mm
- net /OUT3: track 58.9 -> 55.2 mm
- net /OUT5: track 56.9 -> 53.2 mm
- net /OUT1: track 70.5 -> 67.0 mm
- net /OUT2: track 67.6 -> 64.2 mm
- net GND: track 32.8 -> 31.1 mm, vias 34 -> 36
- added copper zone on B.Cu, net +5V
Other:
- board text added: "+"
- board text added: "+12V"
- board text added: "-12V"
- board text added: "3.3V"
- board text added: "5V"
- board text added: "Jonas Norling 2026 Elemental Instruments"
- board text added: "SWD"
- board text removed: "Elemental Instruments Jonas Norling 2026"
