File: hw/vco2/vco2.kicad_sch (KiCad schematic)
At the start: 94 parts, among them Q1 BC847, Q2 BC847, SW1 SW_SPDT, U4 TL072HxD, U5 TL072HxD, U7 TL072HxD, U8 TL072HxD

Commit message: WIP: VCO2 panel
Parts:
- removed TP2: TestPoint_Alt, Holes:TP_0.9mm, symbol Connector:TestPoint_Alt
Changed lines of the file:
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@@
-	)
-	(symbol
-		(lib_id "Connector:TestPoint_Alt")
-		(at 55.88 55.88 270)
-		(mirror x)
-		(unit 1)
-		(exclude_from_sim no)
-		(in_bom yes)
-		(on_board yes)
-		(dnp no)
-		(property "Reference" "TP2"
-			(at 60.4521 58.42 0)
-			(effects
-				(font
-					(size 1.27 1.27)
-				)
-				(justify right)
-			)
-		)
-		(property "Value" "TestPoint_Alt"
-			(at 57.9121 58.42 0)
-			(effects
-				(font
-					(size 1.27 1.27)
-				)
-				(justify right)
-				(hide yes)
-			)
-		)
-		(property "Footprint" "Holes:TP_0.9mm"
-			(at 55.88 50.8 0)
-			(effects
-				(font
-					(size 1.27 1.27)
-				)
-				(hide yes)
-			)
-		)
-		(property "Datasheet" "~"
-			(at 55.88 50.8 0)
-			(effects
-				(font
-					(size 1.27 1.27)
-				)
-				(hide yes)
-			)
-		)
-		(property "Description" "test point (alternative shape)"
-			(at 55.88 55.88 0)
-			(effects
-				(font
-					(size 1.27 1.27)
-				)
-				(hide yes)
-			)
-		)
-		(pin "1"
-		)
-		(instances
-			(project "vco1"
-				(path "/307302bf-1f04-498b-81c7-0944a093f10d"
-					(reference "TP2")
-					(unit 1)
-				)
-			)
-		)
 	)
 	(symbol

Commit message: VCO2 production work
Parts:
- removed TP7: TestPoint_Alt, Holes:TP_0.9mm, symbol Connector:TestPoint_Alt
- R16, R45: value 250k -> 267k
- R31, R39: value 10k -> 4k3
- RV_PWM1, RV_PWM2, RV_RANGE1, RV_RANGE2, RV_TUNE1, RV_TUNE2: value 20k -> 10k
- U4, U5, U7, U8: LCSC (none) -> C4370389
Connections:
- net BACKPLANE_CV: no longer names the net of J_CV1.TN
- no-connect marks 13 -> 14
Changed lines of the file:
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@@
 	)
 	(no_connect
+		(at 31.75 78.74)
+	)
+	(no_connect
 		(at 31.75 124.46)
 	)
@@
 	(wire
 		(pts
-			(xy 33.02 71.12) (xy 33.02 78.74)
-		)
-		(stroke
-			(width 0)
-			(type default)
-		)
-	)
-	(wire
-		(pts
 			(xy 118.11 157.48) (xy 118.11 181.61)
 		)
@@
 	(wire
 		(pts
-			(xy 33.02 71.12) (xy 35.56 71.12)
-		)
-		(stroke
-			(width 0)
-			(type default)
-		)
-	)
-	(wire
-		(pts
 			(xy 160.02 40.64) (xy 152.4 40.64)
 		)
@@
 	(wire
 		(pts
-			(xy 33.02 78.74) (xy 31.75 78.74)
-		)
-		(stroke
-			(width 0)
-			(type default)
-		)
-	)
-	(wire
-		(pts
 			(xy 218.44 120.65) (xy 218.44 111.76)
 		)
@@
 		)
 	)
-	(global_label "BACKPLANE_CV"
-		(shape input)
-		(at 35.56 71.12 0)
-		(fields_autoplaced yes)
-		(effects
-			(font
-				(size 1.27 1.27)
-			)
-			(justify left)
-		)
-		(property "Intersheetrefs" "${INTERSHEET_REFS}"
-			(at 52.6362 71.12 0)
-			(effects
-				(font
-					(size 1.27 1.27)
-				)
-				(justify left)
-				(hide yes)
-			)
-		)
-	)
 	(symbol
 		(lib_id "power:-12V")
@@
 			)
 		)
+		(property "LCSC" "C4370389"
+			(at 163.83 78.74 0)
+			(effects
+				(font
+					(size 1.27 1.27)
+				)
+				(hide yes)
+			)
+		)
 		(pin "8"
 		)
@@
 			)
 		)
-		(property "Value" "10k"
+		(property "Value" "4k3"
 			(at 29.21 27.9399 0)
 			(effects
@@
 			)
 		)
+		(property "LCSC" "C4370389"
+			(at 163.83 55.88 0)
+			(effects
+				(font
+					(size 1.27 1.27)
+				)
+				(hide yes)
+			)
+		)
 		(pin "5"
 		)
@@
 			)
 		)
+		(property "LCSC" "C4370389"
+			(at 168.91 139.7 0)
+			(effects
+				(font
+					(size 1.27 1.27)
+				)
+				(hide yes)
+			)
+		)
 		(pin "5"
 		)
@@
 			)
 		)
+		(property "LCSC" "C4370389"
+			(at 240.03 101.6 0)
+			(effects
+				(font
+					(size 1.27 1.27)
+				)
+				(hide yes)
+			)
+		)
 		(pin "8"
 		)
@@
 			)
 		)
+		(property "LCSC" "C4370389"
+			(at 240.03 78.74 0)
+			(effects
+				(font
+					(size 1.27 1.27)
+				)
+				(hide yes)
+			)
+		)
 		(pin "8"
 		)
@@
 			)
 		)
-		(property "Value" "20k"
+		(property "Value" "10k"
 			(at 82.55 33.0201 0)
 			(effects
@@
 			)
 		)
+		(property "LCSC" "C4370389"
+			(at 240.03 31.75 0)
+			(effects
+				(font
+					(size 1.27 1.27)
+				)
+				(hide yes)
+			)
+		)
 		(pin "5"
 		)
@@
 			)
 		)
+		(property "LCSC" "C4370389"
+			(at 163.83 31.75 0)
+			(effects
+				(font
+					(size 1.27 1.27)
+				)
+				(hide yes)
+			)
+		)
 		(pin "5"
 		)
@@
 			)
 		)
-		(property "Value" "20k"
+		(property "Value" "10k"
 			(at 24.13 54.6101 0)
 			(effects
@@
 			)
 		)
-		(property "Value" "250k"
+		(property "Value" "267k"
 			(at 104.14 52.07 90)
 			(effects
@@
 			)
 		)
-		(property "Value" "20k"
+		(property "Value" "10k"
 			(at 82.55 54.6101 0)
 			(effects
@@
 			)
 		)
-		(property "Value" "10k"
+		(property "Value" "4k3"
 			(at 87.63 27.9399 0)
 			(effects
@@
 			)
 		)
+		(property "LCSC" "C4370389"
+			(at 163.83 101.6 0)
+			(effects
+				(font
+					(size 1.27 1.27)
+				)
+				(hide yes)
+			)
+		)
 		(pin "8"
 		)
@@
 			)
 		)
+		(property "LCSC" "C4370389"
+			(at 240.03 55.88 0)
+			(effects
+				(font
+					(size 1.27 1.27)
+				)
+				(hide yes)
+			)
+		)
 		(pin "5"
 		)
@@
 			)
 		)
+		(property "LCSC" "C4370389"
+			(at 245.11 139.7 0)
+			(effects
+				(font
+					(size 1.27 1.27)
+				)
+				(hide yes)
+			)
+		)
 		(pin "5"
 		)
@@
 			)
 		)
+		(property "LCSC" "C4370389"
+			(at 265.43 139.7 0)
+			(effects
+				(font
+					(size 1.27 1.27)
+				)
+				(hide yes)
+			)
+		)
 		(pin "8"
 		)
@@
 			)
 		)
+		(property "LCSC" "C4370389"
+			(at 189.23 139.7 0)
+			(effects
+				(font
+					(size 1.27 1.27)
+				)
+				(hide yes)
+			)
+		)
 		(pin "8"
 		)
@@
 			)
 		)
-		(property "Value" "20k"
+		(property "Value" "10k"
 			(at 82.55 158.7499 0)
 			(effects
@@
 			)
 		)
-		(property "Value" "20k"
+		(property "Value" "10k"
 			(at 24.13 158.7499 0)
 			(effects
@@
 			)
 		)
-		(property "Value" "20k"
+		(property "Value" "10k"
 			(at 24.13 33.0201 0)
 			(effects
@@
 	)
 	(symbol
-		(lib_id "Connector:TestPoint_Alt")
-		(at 114.3 55.88 270)
-		(mirror x)
-		(unit 1)
-		(exclude_from_sim no)
-		(in_bom yes)
-		(on_board yes)
-		(dnp no)
-		(property "Reference" "TP7"
-			(at 118.8721 58.42 0)
-			(effects
-				(font
-					(size 1.27 1.27)
-				)
-				(justify right)
-			)
-		)
-		(property "Value" "TestPoint_Alt"
-			(at 116.3321 58.42 0)
-			(effects
-				(font
-					(size 1.27 1.27)
-				)
-				(justify right)
-				(hide yes)
-			)
-		)
-		(property "Footprint" "Holes:TP_0.9mm"
-			(at 114.3 50.8 0)
-			(effects
-				(font
-					(size 1.27 1.27)
-				)
-				(hide yes)
-			)
-		)
-		(property "Datasheet" "~"
-			(at 114.3 50.8 0)
-			(effects
-				(font
-					(size 1.27 1.27)
-				)
-				(hide yes)
-			)
-		)
-		(property "Description" "test point (alternative shape)"
-			(at 114.3 55.88 0)
-			(effects
-				(font
-					(size 1.27 1.27)
-				)
-				(hide yes)
-			)
-		)
-		(pin "1"
-		)
-		(instances
-			(project "vco2"
-				(path "/307302bf-1f04-498b-81c7-0944a093f10d"
-					(reference "TP7")
-					(unit 1)
-				)
-			)
-		)
-	)
-	(symbol
 		(lib_id "Device:R")
 		(at 163.83 40.64 270)
@@
 			)
 		)
-		(property "Value" "250k"
+		(property "Value" "267k"
 			(at 45.72 52.07 90)
 			(effects
