File: hw/vco2/vco2.kicad_sch (KiCad schematic)
At the start: 92 parts, among them Q1 BC847, Q2 BC847, SW1 SW_SPDT, U4 TL072HxD, U5 TL072HxD, U7 TL072HxD, U8 TL072HxD

Commit message: VCO2 rev 2 as sent for production at JLCPCB
Parts:
- Q1, Q2: LCSC (none) -> C2145
- U4: LCSC C4370389 -> C6961
Changed lines of the file:
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@@
 			)
 		)
+		(property "LCSC" "C2145"
+			(at 78.74 121.92 0)
+			(effects
+				(font
+					(size 1.27 1.27)
+				)
+				(hide yes)
+			)
+		)
 		(pin "3"
 		)
@@
 			)
 		)
-		(property "LCSC" "C4370389"
+		(property "LCSC" "C6961"
 			(at 163.83 55.88 0)
 			(effects
@@
 			)
 		)
-		(property "LCSC" "C4370389"
+		(property "LCSC" "C6961"
 			(at 168.91 139.7 0)
 			(effects
@@
 			)
 		)
+		(property "LCSC" "C2145"
+			(at 96.52 121.92 0)
+			(effects
+				(font
+					(size 1.27 1.27)
+				)
+				(hide yes)
+			)
+		)
+		(property "Field8" ""
+			(at 96.52 121.92 0)
+			(effects
+				(font
+					(size 1.27 1.27)
+				)
+				(hide yes)
+			)
+		)
 		(pin "3"
 		)
@@
 			)
 		)
-		(property "LCSC" "C4370389"
+		(property "LCSC" "C6961"
 			(at 163.83 31.75 0)
 			(effects
