File: hw/brainboard/mcu.kicad_sch (KiCad schematic)
At the start: 18 parts, among them J1 USB_B_Micro, J2 Conn_ST_STDC14, U3 STM32G474CCTx, Y1 12.288 MHz

Commit message: Laying out brains board
Parts:
- removed C20: 100n, Capacitor_SMD:C_0402_1005Metric, symbol Device:C
- removed TP3: TestPoint, TestPoint:TestPoint_THTPad_D1.0mm_Drill0.5mm, symbol Connector:TestPoint
- added C56: 100n, Capacitor_SMD:C_0402_1005Metric, symbol Device:C
- added D8: LED, LED_SMD:LED_0603_1608Metric, symbol Device:LED
- added R37: 0, Resistor_SMD:R_0402_1005Metric, symbol Device:R
- added R39: 1k, Resistor_SMD:R_0603_1608Metric, symbol Device:R
- added SW1: SW_Push, Button_Switch_SMD:SW_SPST_TS-1088-xR025, symbol Switch:SW_Push
- added U1: APS6404L-3SQRx-SN, Package_SO:SOIC-8_3.9x4.9mm_P1.27mm, symbol Memory_RAM:APS6404L-3SQRx-SN
- J2: footprint Connector_PinHeader_1.27mm:PinHeader_2x07_P1.27mm_Vertical_SMD -> Connector_PinHeader_1.27mm:PinHeader_2x07_P1.27mm_Vertical
- R5: value R -> 10k
Connections:
- net +3.3V: now also C19.1, C56.1, R37.2, SW1.2, U1.8 (VDD)
- net +3.3VA: no longer C19.1
- net BOOT0: now also D8.2 (A), SW1.1
- net GND: now also C56.2, R39.1, U1.4 (VSS)
- net GPIO1: now reaches U3.15 (PA7)
- net GPIO5: now reaches U3.2 (PC13)
- net GPIO6: now reaches U3.3 (PC14)
- net GPIO2: now reaches U3.39 (PA15)
- net GPIO7: now reaches U3.4 (PC15)
- net GPIO3: now reaches U3.41 (PB4)
- net GPIO4: now reaches U3.46 (PB9)
- net QSPI_CLK renamed SPI_CLK
- net SPI_CLK: now also U1.6 (SCLK)
- net QSPI_IO0 renamed SPI_IO0
- net SPI_IO0: now also U1.5 (SI/SIO0)
- net QSPI_IO1 renamed SPI_IO1
- net SPI_IO1: now also U1.2 (SO/SIO1)
- net QSPI_NCS renamed SPI_NCS
- net SPI_NCS: now also U1.1 (~{CE})
- net RX renamed UART_RX
- net TX renamed UART_TX
- new net: D8.1 (K), R39.2
- new net: R37.1, U1.3 (SIO2), U1.7 (SIO3)
Other:
- note added: "BOOT0 low: boot from flash BOOT0 high: boot ROM bootloader Hope this LED circuit will be fine even if we shine a light on it."
- note added: "SPI PSRAM or flash 2 data pins available on the MCU for SPI or dual SPI"
- note added: "decouple VDDA and VREF"
- note removed: "FIXME: - I2S audio - ADC ins - DAC outs - SPI RAM? - BOOT0 button? - MIDI I/O. DNP. - Spare GPIOs for LEDs and buttons"
- moved on the sheet: C10, C12, C13, R5, U3

Commit message: Maybe finished Brain board PCB
Parts:
- C11, C9: value p -> 20p
- J1: LCSC (none) -> C132562
- U1: LCSC (none) -> C5360304; now not fitted
- Y1: footprint Crystal:Crystal_SMD_3225-4Pin_3.2x2.5mm_HandSoldering -> Components:Crystal_SMD_3225-4Pin_3.2x2.5mm_Lagom
Connections:
- net BOOT0: now also R39.2; no longer U3.45 (PB8)
- net GND: now also D8.1 (K); no longer R39.1
- new net: R39.1, U3.45 (PB8)
Other:
- moved on the sheet: D8, R39, R5, SW1
