File: hw/brainboard/supply.kicad_sch (KiCad schematic)
At the start: 23 parts, among them U10 AP130-33Y

Commit message: Laying out brains board
Parts:
- removed U10: AP130-33Y, Package_TO_SOT_SMD:SOT-89-3, symbol Regulator_Linear:AP130-33Y
- added C20, C62, C63: 10u elyt, Capacitor_THT:CP_Radial_D5.0mm_P2.50mm, symbol Device:C_Polarized
- added C57: 2.2u, Capacitor_SMD:C_0603_1608Metric, symbol Device:C
- added D9: LED, LED_SMD:LED_0603_1608Metric, symbol Device:LED
- added R38: 1k, Resistor_SMD:R_0603_1608Metric, symbol Device:R
- added U10: HT7533-1-SOT89, Package_TO_SOT_SMD:SOT-89-3, symbol Regulator_Linear:HT75xx-1-SOT89
- added U11: XC6206P332MR, Package_TO_SOT_SMD:SOT-23-3, symbol Regulator_Linear:XC6206PxxxMR
- added U2: L78L05_SOT89, Package_TO_SOT_SMD:SOT-89-3, symbol Regulator_Linear:L78L05_SOT89
- C1, C2, C7, C8: footprint Capacitor_THT:CP_Radial_D5.0mm_P2.50mm -> Capacitor_SMD:C_0805_2012Metric
- D4, D5, R1, R2: now not fitted
- JP1: footprint Jumper:SolderJumper-2_P1.3mm_Open_RoundedPad1.0x1.5mm -> Jumper:SolderJumper-2_P1.3mm_Open_Pad1.0x1.5mm
Connections:
- net +12V: now also C20.1, U10.2 (VIN), U2.3 (IN)
- net +3.3V: now also U10.3 (VOUT)
- net +3.3VA: now also U11.2 (VO)
- net -12V: now also C62.2
- net GND: now also C20.2, C57.2, C62.1, C63.2, R38.2, U10.1 (GND), U11.1 (GND), U2.2 (GND)
- new net: D9.1 (K), R38.1
- new net +5V: C57.1, C63.1, D9.2 (A), U11.3 (VI), U2.1 (OUT)
Other:
- note added: "HT7533-1 and XC6206P332MR are JLCPCB basic parts how bad can they be?"
- note removed: "FIXME: Find good 16V tolerant parts Marbles uses "R-78E3.3-0.5" (DCDC module) for digital and LD2981ABU33 (SOT-89) for analog."
- note removed: "FIXME: No, now we need 5V"
- moved on the sheet: C1, C2, C3, C4, C5, C6, C7, C8, D1, D2, D3, D6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

Commit message: Maybe finished Brain board PCB
Parts:
- removed D4, D5, D9: LED, LED_SMD:LED_0603_1608Metric, symbol Device:LED
- removed R1, R2: 2k2, Resistor_SMD:R_0603_1608Metric, symbol Device:R
- removed R38: 1k, Resistor_SMD:R_0603_1608Metric, symbol Device:R
- C7, C8: now fitted
