File: hw/brainboard/audio_io.kicad_sch (KiCad schematic)
At the start: 21 parts, among them U4 TL074

Commit message: Laying out brains board
Parts:
- removed C25, C26: 100n, Capacitor_SMD:C_0402_1005Metric, symbol Device:C

Commit message: Maybe finished Brain board PCB
Parts:
- U4: LCSC (none) -> C6964
Changed lines of the file:
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@@
+			)
+		)
+		(property "LCSC" "C6964"
+			(at 138.43 97.79 0)
+			(effects
+				(font
+					(size 1.27 1.27)
+				)
+				(hide yes)
+			)
+		)
+		(property "Field6" ""
+			(at 138.43 97.79 0)
+			(effects
+				(font
+					(size 1.27 1.27)
+				)
+				(hide yes)
 			)
 		)
@@
 			)
 		)
+		(property "LCSC" "C6964"
+			(at 138.43 120.65 0)
+			(effects
+				(font
+					(size 1.27 1.27)
+				)
+				(hide yes)
+			)
+		)
+		(property "Field6" ""
+			(at 138.43 120.65 0)
+			(effects
+				(font
+					(size 1.27 1.27)
+				)
+				(hide yes)
+			)
+		)
 		(pin "13"
 		)
@@
 			)
 		)
+		(property "LCSC" "C6964"
+			(at 129.54 175.26 0)
+			(effects
+				(font
+					(size 1.27 1.27)
+				)
+				(hide yes)
+			)
+		)
+		(property "Field6" ""
+			(at 129.54 175.26 0)
+			(effects
+				(font
+					(size 1.27 1.27)
+				)
+				(hide yes)
+			)
+		)
 		(pin "2"
 		)
@@
 		)
 		(property "Description" "Quad Low-Noise JFET-Input Operational Amplifiers, DIP-14/SOIC-14"
+			(at 138.43 50.8 0)
+			(effects
+				(font
+					(size 1.27 1.27)
+				)
+				(hide yes)
+			)
+		)
+		(property "LCSC" "C6964"
+			(at 138.43 50.8 0)
+			(effects
+				(font
+					(size 1.27 1.27)
+				)
+				(hide yes)
+			)
+		)
+		(property "Field6" ""
 			(at 138.43 50.8 0)
 			(effects
@@
 			(at 138.43 74.93 0)
 			(effects
+				(font
+					(size 1.27 1.27)
+				)
+				(hide yes)
+			)
+		)
+		(property "LCSC" "C6964"
+			(at 138.43 74.93 0)
+			(effects
+				(font
+					(size 1.27 1.27)
+				)
+				(hide yes)
+			)
+		)
+		(property "Field6" ""
+			(at 138.43 74.93 0)
+			(effects

Commit message: Brainboard polishing
Parts:
- R10, R11, R8, R9: value 39k -> 100k
- R12, R13, R6, R7: value 10k -> 15k
Other:
- note added: "2.1VRMS ground centered = 3Vpp"
- note added: "20Vpp (±10V)"
- note added: "3.0Vpp centered on 2.5V"
Changed lines of the file:
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@@
 	(generator_version "9.0")
 	(paper "A4")
+	(text "20Vpp (±10V)"
+		(exclude_from_sim no)
+		(at 97.282 110.744 0)
+		(effects
+			(font
+				(size 1.27 1.27)
+			)
+		)
+	)
+	(text "20Vpp (±10V)"
+		(exclude_from_sim no)
+		(at 173.228 61.976 0)
+		(effects
+			(font
+				(size 1.27 1.27)
+			)
+		)
+	)
+	(text "3.0Vpp centered on 2.5V"
+		(exclude_from_sim no)
+		(at 181.864 106.934 0)
+		(effects
+			(font
+				(size 1.27 1.27)
+			)
+		)
+	)
+	(text "2.1VRMS ground centered = 3Vpp"
+		(exclude_from_sim no)
+		(at 84.328 62.484 0)
+		(effects
+			(font
+				(size 1.27 1.27)
+				(thickness 0.1588)
+			)
+			(justify left)
+		)
+	)
 	(junction
 		(at 148.59 97.79)
@@
 			)
 		)
-		(property "Value" "10k"
+		(property "Value" "15k"
 			(at 138.43 102.87 90)
 			(effects
@@
 			)
 		)
-		(property "Value" "10k"
+		(property "Value" "15k"
 			(at 120.65 73.66 90)
 			(effects
@@
 			)
 		)
-		(property "Value" "39k"
+		(property "Value" "100k"
 			(at 120.65 96.52 90)
 			(effects
@@
 			)
 		)
-		(property "Value" "39k"
+		(property "Value" "100k"
 			(at 138.43 80.01 90)
 			(effects
@@
 			)
 		)
-		(property "Value" "39k"
+		(property "Value" "100k"
 			(at 120.65 119.38 90)
 			(effects
@@
 			)
 		)
-		(property "Value" "10k"
+		(property "Value" "15k"
 			(at 120.65 49.53 90)
 			(effects
@@
 			)
 		)
-		(property "Value" "10k"
+		(property "Value" "15k"
 			(at 138.43 125.73 90)
 			(effects
@@
 			)
 		)
-		(property "Value" "39k"
+		(property "Value" "100k"
 			(at 138.43 55.88 90)
 			(effects
