File: hw/brainboard/brainboard.kicad_pcb (KiCad board)
At the start: 2 copper layers, 110 parts, among them J1 USB_B_Micro, J2 Conn_ST_STDC14, U10 AP130-33Y, U3 STM32G474CCTx, U4 TL074, U5 PCM1808, U6 LM4040DBZ-10, U7 TLV2372, U8 TLV2372, U9 PCM5102A

Commit message: Laying out brains board
Parts:
- removed TP3: TestPoint, TestPoint:TestPoint_THTPad_D1.0mm_Drill0.5mm
- added C56: 100n, Capacitor_SMD:C_0402_1005Metric, B.Cu at (39.5, 68.9)
- added C57: 2.2u, Capacitor_SMD:C_0603_1608Metric, F.Cu at (60.5, 117.0)
- added C58: 100n, Capacitor_SMD:C_0402_1005Metric, F.Cu at (53.0, 80.5)
- added C59: 100n, Capacitor_SMD:C_0402_1005Metric, F.Cu at (64.0, 80.5)
- added C60: 1n, Capacitor_SMD:C_0402_1005Metric, F.Cu at (53.0, 74.5)
- added C61: 100n, Capacitor_SMD:C_0402_1005Metric, F.Cu at (64.0, 79.5)
- added C62: 10u elyt, Capacitor_THT:CP_Radial_D5.0mm_P2.50mm, B.Cu at (85.5, 100.7)
- added C63: 10u elyt, Capacitor_THT:CP_Radial_D5.0mm_P2.50mm, B.Cu at (90.2, 91.0)
- added D8: LED, LED_SMD:LED_0603_1608Metric, F.Cu at (75.5, 96.5)
- added D9: LED, LED_SMD:LED_0603_1608Metric, B.Cu at (24.5, 114.0)
- added J3: gpio, Connector_PinHeader_2.54mm:PinHeader_1x10_P2.54mm_Vertical, F.Cu at (53.0, 145.0)
- added J4: misc, Connector_PinHeader_2.54mm:PinHeader_1x10_P2.54mm_Vertical, F.Cu at (53.0, 54.5)
- added J5: inputs, Connector_PinHeader_2.54mm:PinHeader_1x10_P2.54mm_Vertical, F.Cu at (53.0, 147.5)
- added J6: audio_dac_power, Connector_PinHeader_2.54mm:PinHeader_1x10_P2.54mm_Vertical, F.Cu at (53.0, 52.0)
- added J7: eurorack_power, Connector_IDC:IDC-Header_2x05_P2.54mm_Vertical, F.Cu at (75.0, 119.1)
- added R37: 0, Resistor_SMD:R_0402_1005Metric, B.Cu at (34.5, 70.9)
- added R38: 1k, Resistor_SMD:R_0603_1608Metric, B.Cu at (24.5, 115.5)
- added R39: 1k, Resistor_SMD:R_0603_1608Metric, F.Cu at (75.5, 93.5)
- added R40: 33k, Resistor_SMD:R_0603_1608Metric, F.Cu at (52.5, 83.5)
- added R41: 1k, Resistor_SMD:R_0603_1608Metric, F.Cu at (52.5, 85.0)
- added R42: 33k, Resistor_SMD:R_0603_1608Metric, F.Cu at (64.5, 83.0)
- added R43: 100k, Resistor_SMD:R_0603_1608Metric, F.Cu at (52.5, 82.0)
- added R44: 33k, Resistor_SMD:R_0603_1608Metric, F.Cu at (52.5, 77.5)
- added R45: 1k, Resistor_SMD:R_0603_1608Metric, F.Cu at (52.5, 76.0)
- added R46: 100k, Resistor_SMD:R_0603_1608Metric, F.Cu at (64.5, 84.5)
- added R47: 100k, Resistor_SMD:R_0603_1608Metric, F.Cu at (52.5, 79.0)
- added R48: ??, Resistor_SMD:R_0603_1608Metric, F.Cu at (64.5, 78.0)
- added R49: ??, Resistor_SMD:R_0603_1608Metric, F.Cu at (64.5, 76.5)
- added R50: 1k, Resistor_SMD:R_0603_1608Metric, F.Cu at (64.5, 86.0)
- added SW1: SW_Push, Button_Switch_SMD:SW_SPST_TS-1088-xR025, F.Cu at (72.0, 95.0)
- added TP1: 3V, Holes:TP_0.9mm, F.Cu at (40.1, 111.4)
- added TP2: 3VA, Holes:TP_0.9mm, F.Cu at (40.1, 113.8)
- added U1: APS6404L-3SQRx-SN, Package_SO:SOIC-8_3.9x4.9mm_P1.27mm, B.Cu at (39.5, 72.4)
- added U11: XC6206P332MR, Package_TO_SOT_SMD:SOT-23-3, F.Cu at (54.0, 119.0)
- added U12: TL074, Package_SO:SOIC-14_3.9x8.7mm_P1.27mm, F.Cu at (58.5, 80.5)
- added U2: L78L05_SOT89, Package_TO_SOT_SMD:SOT-89-3, F.Cu at (64.0, 115.5)
- added Y1: 12.288 MHz, Crystal:Crystal_SMD_3225-4Pin_3.2x2.5mm_HandSoldering, F.Cu at (66.0, 97.0)
- C1, C2, C7, C8: footprint Capacitor_THT:CP_Radial_D5.0mm_P2.50mm -> Capacitor_SMD:C_0805_2012Metric
- C11, C9: footprint Capacitor_SMD:C_0603_1608Metric -> Capacitor_SMD:C_0402_1005Metric
- C19, D4, D5, R1, R2: moved to B.Cu
- C20: value 100n -> 10u elyt; footprint Capacitor_SMD:C_0402_1005Metric -> Capacitor_THT:CP_Radial_D5.0mm_P2.50mm; moved to B.Cu
- C25, C26: value 100n -> 1n
- J2: footprint Connector_PinHeader_1.27mm:PinHeader_2x07_P1.27mm_Vertical_SMD -> Connector_PinHeader_1.27mm:PinHeader_2x07_P1.27mm_Vertical
- JP1: footprint Jumper:SolderJumper-2_P1.3mm_Open_RoundedPad1.0x1.5mm -> Jumper:SolderJumper-2_P1.3mm_Open_Pad1.0x1.5mm
- R5: value R -> 10k
- U10: value AP130-33Y -> HT7533-1-SOT89
- moved C32 129.6 mm to (53.5, 139.0), turned to 90 degrees
- moved R27 127.9 mm to (55.0, 139.5), turned to 90 degrees
- moved C30 125.4 mm to (54.0, 128.0), turned to 90 degrees
- moved C33 121.7 mm to (55.0, 128.0), turned to -90 degrees
- moved R23 120.8 mm to (58.0, 139.5), turned to -90 degrees
- moved R28 117.4 mm to (58.0, 127.5), turned to 90 degrees
- moved R19 117.3 mm to (56.5, 139.5), turned to 90 degrees
- moved R24 113.9 mm to (56.5, 127.5), turned to -90 degrees
- moved C34 113.4 mm to (70.5, 139.0), turned to 90 degrees
- moved C24 112.3 mm to (58.0, 59.0), turned to -90 degrees
- moved C29 110.8 mm to (66.0, 136.0), turned to 90 degrees
- moved U7 110.4 mm to (56.5, 133.5), turned to 90 degrees
- moved R13 110.3 mm to (53.5, 58.5), turned to 90 degrees
- moved R18 110.3 mm to (64.5, 136.0), turned to -90 degrees
- moved R29 110.2 mm to (73.5, 139.5), turned to -90 degrees
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Connections:
- net Net-(U5-VREF) renamed /codec/VREF_DECOUPLE
- C19 pad 1: +3.3VA -> +3.3V
- C20 pad 1: +3.3VA -> +12V
- C25 pad 1: +12V -> Net-(U12C--)
- C25 pad 2: GND -> /DAC3
- C26 pad 1: GND -> Net-(U12B--)
- C26 pad 2: -12V -> Net-(C26-Pad2)
- C36 pad 1: /codec/AUDIO_OUT_L -> /audio_io/DAC_L
- C37 pad 1: /codec/AUDIO_OUT_R -> /audio_io/DAC_R
- C48 pad 1: /codec/AUDIO_IN_L -> /audio_io/ADC_L
- C49 pad 1: /codec/AUDIO_IN_R -> /audio_io/ADC_R
- D1 pad 2: /supply/USB_VBUS -> /VBUS
- D2 pad 2: /supply/+12V_IN -> /+12V
- D3 pad 1: /supply/-12V_IN -> /-12V
- J1 pad 1: /mcu/USB_VBUS -> /VBUS
- R33 pad 1: /codec/AUDIO_OUT_L -> /audio_io/DAC_L
- R34 pad 1: /codec/AUDIO_OUT_R -> /audio_io/DAC_R
- U10 pad 1: +3.3VA -> GND
- U10 pad 2: GND -> +12V
- U10 pad 3: +12V -> +3.3V
- U3 pad 12: /mcu/AOUT1 -> /AOUT1
- U3 pad 13: /mcu/AOUT2 -> /AOUT2
- U3 pad 14: /mcu/AOUT3 -> /AOUT3
- U3 pad 15: unconnected-(U3-PA7-Pad15) -> /mcu/GPIO1
- U3 pad 2: unconnected-(U3-PC13-Pad2) -> /mcu/GPIO5
- U3 pad 26: /mcu/AIN5 -> /analog_io/CV_INT1
- U3 pad 27: /mcu/AIN6 -> /analog_io/CV_INT2
- U3 pad 28: /mcu/AIN7 -> /analog_io/CV_INT3
- U3 pad 29: /mcu/AIN8 -> /analog_io/CV_INT4
- U3 pad 3: unconnected-(U3-PC14-Pad3) -> /mcu/GPIO6
- U3 pad 30: /mcu/I2S_BCLK -> /codec/BCK
- U3 pad 31: /mcu/I2S_LRCLK -> /codec/LRCK
- U3 pad 32: /mcu/I2S_DOUT -> /codec/DIN
- U3 pad 39: unconnected-(U3-PA15-Pad39) -> /mcu/GPIO2
- U3 pad 4: unconnected-(U3-PC15-Pad4) -> /mcu/GPIO7
- U3 pad 41: unconnected-(U3-PB4-Pad41) -> /mcu/GPIO3
- U3 pad 42: /mcu/I2S_DIN -> /codec/DOUT
- U3 pad 46: unconnected-(U3-PB9-Pad46) -> /mcu/GPIO4
Other:
- board outline added: 29 x 100 mm
- board text added: "Analog CV in"
- board text added: "Audio ADC"
- board text added: "Audio DAC"
- board text added: "Audio amp"
- board text added: "DAC amp"
- board text added: "MCU"
- board text added: "Power"

Commit message: Maybe finished Brain board PCB
Parts:
- removed D4, D5, D9: LED, LED_SMD:LED_0603_1608Metric
- removed R1, R2: 2k2, Resistor_SMD:R_0603_1608Metric
- removed R38: 1k, Resistor_SMD:R_0603_1608Metric
- added G***: LOGO, elemental:elemental-4mm, F.Cu at (68.1, 84.9)
- added G***: LOGO, elemental:elemental-25.4mm, B.Cu at (64.5, 60.6)
- added H1: MountingHole, Holes:MountingHole_3.2mm_M3_Pad, F.Cu at (74.0, 86.5)
- added TP10: I2S, Holes:TP_0.8mm_pad, B.Cu at (70.0, 92.0)
- added TP11: ADC_L, Holes:TP_0.9mm, B.Cu at (70.0, 65.0)
- added TP12: ADC_R, Holes:TP_0.9mm, B.Cu at (68.0, 65.0)
- added TP3: -10V, Holes:TP_0.8mm_pad, B.Cu at (65.0, 138.0)
- added TP4: DAC_L, Holes:TP_0.9mm, B.Cu at (62.0, 75.0)
- added TP5: DAC_R, Holes:TP_0.9mm, B.Cu at (62.0, 73.0)
- added TP6: I2S, Holes:TP_0.8mm_pad, B.Cu at (71.0, 92.0)
- added TP7: I2S, Holes:TP_0.8mm_pad, B.Cu at (72.0, 92.0)
- added TP8: I2S, Holes:TP_0.8mm_pad, B.Cu at (68.0, 92.0)
- added TP9: I2S, Holes:TP_0.8mm_pad, B.Cu at (69.0, 92.0)
- C11, C9: value p -> 20p
- C19, C20, C56, C62, C63, R37, U1: moved to F.Cu
- JP1: moved to B.Cu
- R36: footprint Resistor_SMD:R_0402_1005Metric -> Resistor_SMD:R_0603_1608Metric
- R48: value ?? -> 160k
- R49: value ?? -> 100k
- Y1: footprint Crystal:Crystal_SMD_3225-4Pin_3.2x2.5mm_HandSoldering -> Components:Crystal_SMD_3225-4Pin_3.2x2.5mm_Lagom
- moved R37 54.9 mm to (69.0, 113.5)
- moved C56 49.5 mm to (67.0, 110.0)
- moved C19 49.1 mm to (64.0, 110.0), turned to 180 degrees
- moved U1 47.9 mm to (64.0, 113.5), turned to 0 degrees
- moved TP2 33.5 mm to (70.0, 129.0), turned to 180 degrees
- moved C63 33.4 mm to (72.0, 119.0)
- moved TP1 32.2 mm to (62.0, 135.0), turned to 180 degrees
- moved JP1 29.0 mm to (67.0, 129.0), turned to 180 degrees
- moved C62 23.7 mm to (75.0, 122.0), turned to 0 degrees
- moved C20 22.7 mm to (72.0, 125.0), turned to 180 degrees
- moved C42 21.6 mm to (78.0, 69.0), turned to 90 degrees
- moved C44 21.2 mm to (70.5, 69.0), turned to 90 degrees
- moved C38 20.1 mm to (75.0, 69.0), turned to 90 degrees
- moved C41 20.1 mm to (73.5, 69.0), turned to 90 degrees
- moved C43 19.7 mm to (76.5, 69.5), turned to 90 degrees
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Connections:
- C26 pad 2: Net-(C26-Pad2) -> /DAC2
- C60 pad 2: Net-(C60-Pad2) -> /DAC1
- D8 pad 1: Net-(D8-K) -> GND
- J3 pad 8: unconnected-(J3-Pin_8-Pad8) -> /+12V
- J3 pad 9: unconnected-(J3-Pin_9-Pad9) -> /-12V
- R39 pad 1: GND -> Net-(U3-PB8)
- R39 pad 2: Net-(D8-K) -> /mcu/BOOT0
- R43 pad 1: Net-(C26-Pad2) -> /DAC2
- R47 pad 1: Net-(C60-Pad2) -> /DAC1
- U3 pad 11: /mcu/I2S_MCLK -> /codec/MCLK
- U3 pad 45: /mcu/BOOT0 -> Net-(U3-PB8)
Routing:
- net +3.3V: track 0.00 -> 228.7 mm, vias 0 -> 10
- net +3.3VA: track 0.00 -> 178.7 mm, vias 0 -> 8
- net +12V: track 0.00 -> 161.5 mm, vias 0 -> 13
- net -12V: track 0.00 -> 154.2 mm, vias 0 -> 5
- net /+12V: track 0.00 -> 121.1 mm
- net /-12V: track 0.00 -> 106.8 mm
- net /mcu/QSPI_CLK: track 0.00 -> 94.3 mm, vias 0 -> 5
- net /mcu/QSPI_IO0: track 0.00 -> 88.8 mm, vias 0 -> 5
- net +5V: track 0.00 -> 87.4 mm, vias 0 -> 2
- net /mcu/QSPI_NCS: track 0.00 -> 84.2 mm, vias 0 -> 5
- net /mcu/QSPI_IO1: track 0.00 -> 72.5 mm, vias 0 -> 5
- net /mcu/AIN4: track 0.00 -> 69.0 mm, vias 0 -> 2
- net /codec/LRCK: track 0.00 -> 68.3 mm, vias 0 -> 5
- net /analog_io/CV_INT3: track 0.00 -> 66.9 mm, vias 0 -> 2
- net /codec/BCK: track 0.00 -> 66.1 mm, vias 0 -> 5
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- added copper zone on B.Cu, net +12V
- added copper zone on F.Cu, net +12V
- added copper zone on B.Cu, net GND
- added copper zone on F.Cu, net GND
- added copper zone on In1.Cu, net GND
- added copper zone on In2.Cu, net GND
Other:
- outline, holes or cut-outs redrawn
- copper layers 2 -> 4
- board text added: "+"
- board text added: "+12V ·"
- board text added: "-10V"
- board text added: "-12V ·"
- board text added: "3.3VA ·"
- board text added: "5V ·"
- board text added: "Eurorack Brainboard"
- board text added: "Eurorack Brainboard rev. 1"
- board text added: "JN 2026"
- board text added: "Jonas Norling 2026"
- board text added: "rev. 1"
- board text added: "· 3.3V"

Commit message: Brainboard polishing
Parts:
- removed C48, C49: 1u, Capacitor_SMD:C_0603_1608Metric
- R10, R11, R8, R9: value 39k -> 100k
- R12, R13, R6, R7: value 10k -> 15k
- moved G*** 0.38 mm to (68.1, 85.2)
Connections:
- TP11 pad 1: Net-(U5-VINL) -> /audio_io/ADC_L
- TP12 pad 1: Net-(U5-VINR) -> /audio_io/ADC_R
- U5 pad 13: Net-(U5-VINL) -> /audio_io/ADC_L
- U5 pad 14: Net-(U5-VINR) -> /audio_io/ADC_R
Routing:
- net /audio_io/ADC_L: track 2.84 -> 10.8 mm
- net Net-(U5-VINL): track 7.14 -> 0.00 mm
- net /audio_io/ADC_R: track 12.2 -> 18.5 mm
- net Net-(U5-VINR): track 4.79 -> 0.00 mm
- net GND: vias 129 -> 131
Other:
- board size 29 x 100 mm -> 29 x 99.5 mm
- board text added: "+12"
- board text added: "+12 CV3"
- board text added: "-12"
- board text added: "3.3"
- board text added: "AO1"
- board text added: "AO2"
- board text added: "AO3"
- board text added: "CV4"
- board text added: "GND"
- board text added: "INL"
- board text added: "INR"
- board text added: "IO1 3.3A"
- board text added: "IO2 A1"
- board text added: "IO3 A2"
- board text added: "IO4 A3"
- board text added: "IO5 A4"
- board text added: "IO6 CV1"
- board text added: "IO7 CV2"
- board text added: "OL"
- board text added: "OR"
