File: hw/brainboard/brainboard.kicad_sch (KiCad schematic)
At the start: 0 parts

Commit message: Laying out brains board
Parts:
- added J3: gpio, Connector_PinHeader_2.54mm:PinHeader_1x10_P2.54mm_Vertical, symbol Connector:Conn_01x10_Pin
- added J4: misc, Connector_PinHeader_2.54mm:PinHeader_1x10_P2.54mm_Vertical, symbol Connector:Conn_01x10_Pin
- added J5: inputs, Connector_PinHeader_2.54mm:PinHeader_1x10_P2.54mm_Vertical, symbol Connector:Conn_01x10_Pin
- added J6: audio_dac_power, Connector_PinHeader_2.54mm:PinHeader_1x10_P2.54mm_Vertical, symbol Connector:Conn_01x10_Pin
- added J7: eurorack_power, Connector_IDC:IDC-Header_2x05_P2.54mm_Vertical, symbol Connector_Generic:Conn_02x05_Odd_Even
Connections:
- net analog_io/CV1: now also J5.6 (Pin_6)
- net analog_io/CV2: now also J5.7 (Pin_7)
- net analog_io/CV3: now also J5.8 (Pin_8)
- net analog_io/CV4: now also J5.9 (Pin_9)
- net audio_io/AUDIO_IN_L: now also J6.4 (Pin_4)
- net audio_io/AUDIO_IN_R: now also J6.5 (Pin_5)
- net audio_io/AUDIO_OUT_L: now also J6.6 (Pin_6)
- net audio_io/AUDIO_OUT_R: now also J6.7 (Pin_7)
- net mcu/AIN1: now also J5.2 (Pin_2)
- net mcu/AIN2: now also J5.3 (Pin_3)
- net mcu/AIN3: now also J5.4 (Pin_4)
- net mcu/AIN4: now also J5.5 (Pin_5)
- new net +12V: J6.8 (Pin_8), J7.10 (Pin_10), J7.9 (Pin_9)
- new net +3.3V: J4.1 (Pin_1)
- new net +3.3VA: J5.1 (Pin_1)
- new net -12V: J6.9 (Pin_9), J7.1 (Pin_1), J7.2 (Pin_2)
- new net DAC1: J6.1 (Pin_1)
- new net DAC2: J6.2 (Pin_2)
- new net DAC3: J6.3 (Pin_3)
- new net GND: J3.10 (Pin_10), J4.10 (Pin_10), J5.10 (Pin_10), J6.10 (Pin_10), J7.3 (Pin_3), J7.4 (Pin_4), J7.5 (Pin_5), J7.6 (Pin_6), J7.7 (Pin_7), J7.8 (Pin_8)
- new net mcu/BOOT0: J4.3 (Pin_3)
- new net mcu/GPIO1: J3.1 (Pin_1)
- new net mcu/GPIO2: J3.2 (Pin_2)
- new net mcu/GPIO3: J3.3 (Pin_3)
- new net mcu/GPIO4: J3.4 (Pin_4)
- new net mcu/GPIO5: J3.5 (Pin_5)
- new net mcu/GPIO6: J3.6 (Pin_6)
- new net mcu/GPIO7: J3.7 (Pin_7)
- new net mcu/NRST: J4.2 (Pin_2)
- new net mcu/SPI_CLK: J4.9 (Pin_9)
- new net mcu/SPI_IO0: J4.7 (Pin_7)
- new net mcu/SPI_IO1: J4.6 (Pin_6)
- new net mcu/SPI_NCS: J4.8 (Pin_8)
- new net mcu/UART_RX: J4.5 (Pin_5)
- new net mcu/UART_TX: J4.4 (Pin_4)
Other:
- sheet analog_io ports: added DAC1, DAC2, DAC3, DAC_INT1, DAC_INT2, DAC_INT3; removed none
- sheet mcu ports: added BOOT0, GPIO1, GPIO2, GPIO3, GPIO4, GPIO5, GPIO6, GPIO7, NRST, SPI_CLK, SPI_IO0, SPI_IO1, SPI_NCS, UART_RX, UART_TX; removed none
- sheet supply ports: added +12V_IN, -12V_IN; removed none

Commit message: Maybe finished Brain board PCB
Parts:
- added H1: MountingHole, Holes:MountingHole_3.2mm_M3_Pad, symbol Mechanical:MountingHole
Connections:
- net +12V: now also J3.8 (Pin_8)
- net -12V: now also J3.9 (Pin_9)
Other:
- sheet codec ports: added MCLK; removed SCK
Changed lines of the file:
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@@
+	(wire
+		(pts
+			(xy 157.48 129.54) (xy 168.91 129.54)
+		)
+		(stroke
+			(width 0)
+			(type default)
+		)
+	)
 	(wire
 		(pts
@@
 		(pts
 			(xy 134.62 127) (xy 168.91 127)
+		)
+		(stroke
+			(width 0)
+			(type default)
+		)
+	)
+	(wire
+		(pts
+			(xy 157.48 132.08) (xy 168.91 132.08)
 		)
 		(stroke
@@
 		)
 	)
+	(label "-12V"
+		(at 157.48 132.08 0)
+		(effects
+			(font
+				(size 1.27 1.27)
+			)
+			(justify left bottom)
+		)
+	)
 	(label "DAC3"
 		(at 220.98 91.44 0)
@@
 			)
 			(justify right bottom)
+		)
+	)
+	(label "+12V"
+		(at 157.48 129.54 0)
+		(effects
+			(font
+				(size 1.27 1.27)
+			)
+			(justify left bottom)
 		)
 	)
@@
 	)
 	(symbol
+		(lib_id "Mechanical:MountingHole")
+		(at 55.88 167.64 0)
+		(unit 1)
+		(exclude_from_sim no)
+		(in_bom no)
+		(on_board yes)
+		(dnp no)
+		(fields_autoplaced yes)
+		(property "Reference" "H1"
+			(at 58.42 166.3699 0)
+			(effects
+				(font
+					(size 1.27 1.27)
+				)
+				(justify left)
+			)
+		)
+		(property "Value" "MountingHole"
+			(at 58.42 168.9099 0)
+			(effects
+				(font
+					(size 1.27 1.27)
+				)
+				(justify left)
+			)
+		)
+		(property "Footprint" "Holes:MountingHole_3.2mm_M3_Pad"
+			(at 55.88 167.64 0)
+			(effects
+				(font
+					(size 1.27 1.27)
+				)
+				(hide yes)
+			)
+		)
+		(property "Datasheet" "~"
+			(at 55.88 167.64 0)
+			(effects
+				(font
+					(size 1.27 1.27)
+				)
+				(hide yes)
+			)
+		)
+		(property "Description" "Mounting Hole without connection"
+			(at 55.88 167.64 0)
+			(effects
+				(font
+					(size 1.27 1.27)
+				)
+				(hide yes)
+			)
+		)
+		(instances
+			(project "brainboard"
+				(path "/c4f877e5-ce69-4e50-ab01-826c8aac2c0b"
+					(reference "H1")
+					(unit 1)
+				)
+			)
+		)
+	)
+	(symbol
 		(lib_id "Connector:Conn_01x10_Pin")
 		(at 234.95 96.52 0)
@@
 			)
 		)
-		(pin "SCK" input
-			(at 160.02 96.52 180)
-			(effects
-				(font
-					(size 1.27 1.27)
-				)
-				(justify left)
-			)
-		)
 		(pin "AUDIO_OUT_R" output
 			(at 184.15 101.6 0)
@@
 			)
 		)
+		(pin "MCLK" input
+			(at 160.02 96.52 180)
+			(effects
+				(font
+					(size 1.27 1.27)
+				)
+				(justify left)
+			)
+		)

Commit message: Brainboard polishing
Other:
- note added: "GPIO5-7 weak outputs"
Changed lines of the file:
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@@
 		(company "Jonas Norling")
+	)
+	(text "GPIO5-7\nweak\noutputs"
+		(exclude_from_sim no)
+		(at 146.812 124.714 0)
+		(effects
+			(font
+				(size 1.27 1.27)
+			)
+			(justify left)
+		)
 	)
 	(wire
