File: hw/brainboard/codec.kicad_sch (KiCad schematic)
At the start: 28 parts, among them U5 PCM1808, U9 PCM5102A

Commit message: Laying out brains board
Connections:
- net VREF_DECOUPLE: now reaches C50.1, C51.1, U5.1 (VREF)
Changed lines of the file:
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@@
+		)
+	)
+	(label "VREF_DECOUPLE"
+		(at 238.76 64.77 0)
+		(effects
+			(font
+				(size 1.27 1.27)
+			)
+			(justify left bottom)
 		)
 	)

Commit message: Maybe finished Brain board PCB
Parts:
- added TP10, TP6, TP7, TP8, TP9: I2S, Holes:TP_0.8mm_pad, symbol Connector:TestPoint
- added TP11: ADC_L, Holes:TP_0.9mm, symbol Connector:TestPoint
- added TP12: ADC_R, Holes:TP_0.9mm, symbol Connector:TestPoint
- added TP4: DAC_L, Holes:TP_0.9mm, symbol Connector:TestPoint
- added TP5: DAC_R, Holes:TP_0.9mm, symbol Connector:TestPoint
- R36: footprint Resistor_SMD:R_0402_1005Metric -> Resistor_SMD:R_0603_1608Metric
Connections:
- net AUDIO_OUT_L: now also TP4.1
- net AUDIO_OUT_R: now also TP5.1
- net BCK: now also TP9.1
- net DIN: now also TP7.1
- net DOUT: now also TP8.1
- net LRCK: now also TP6.1
- net MCLK: now also TP10.1
- net at C48.2, U5.13 (VINL): now also TP11.1
- net at C49.2, U5.14 (VINR): now also TP12.1

Commit message: Brainboard polishing
Parts:
- removed C48, C49: 1u, Capacitor_SMD:C_0603_1608Metric, symbol Device:C
Connections:
- net AUDIO_IN_L: now also TP11.1, U5.13 (VINL)
- net AUDIO_IN_R: now also TP12.1, U5.14 (VINR)
Other:
- note added: "3.0Vp-p centered on 2.5V"
Changed lines of the file:
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@@
+		)
+	)
+	(text "3.0Vp-p centered on 2.5V"
+		(exclude_from_sim no)
+		(at 168.402 93.472 0)
+		(effects
+			(font
+				(size 1.27 1.27)
+			)
 		)
 	)
@@
 	(wire
 		(pts
-			(xy 161.29 87.63) (xy 171.45 87.63)
+			(xy 177.8 87.63) (xy 185.42 87.63)
 		)
 		(stroke
@@
 	(wire
 		(pts
-			(xy 161.29 90.17) (xy 163.83 90.17)
+			(xy 177.8 90.17) (xy 185.42 90.17)
 		)
 		(stroke
@@
 	(wire
 		(pts
-			(xy 179.07 87.63) (xy 185.42 87.63)
-		)
-		(stroke
-			(width 0)
-			(type default)
-		)
-	)
-	(wire
-		(pts
 			(xy 66.04 48.26) (xy 66.04 58.42)
 		)
@@
 		(pts
 			(xy 238.76 64.77) (xy 248.92 64.77)
-		)
-		(stroke
-			(width 0)
-			(type default)
-		)
-	)
-	(wire
-		(pts
-			(xy 171.45 90.17) (xy 185.42 90.17)
 		)
 		(stroke
@@
 	(hierarchical_label "AUDIO_IN_L"
 		(shape input)
-		(at 161.29 87.63 180)
+		(at 177.8 87.63 180)
 		(effects
 			(font
@@
 	(hierarchical_label "AUDIO_IN_R"
 		(shape input)
-		(at 161.29 90.17 180)
+		(at 177.8 90.17 180)
 		(effects
 			(font
@@
 			)
 			(justify left)
-		)
-	)
-	(symbol
-		(lib_id "Device:C")
-		(at 175.26 87.63 90)
-		(unit 1)
-		(exclude_from_sim no)
-		(in_bom yes)
-		(on_board yes)
-		(dnp no)
-		(property "Reference" "C48"
-			(at 173.9899 83.82 0)
-			(effects
-				(font
-					(size 1.27 1.27)
-				)
-				(justify left)
-			)
-		)
-		(property "Value" "1u"
-			(at 176.5299 83.82 0)
-			(effects
-				(font
-					(size 1.27 1.27)
-				)
-				(justify left)
-			)
-		)
-		(property "Footprint" "Capacitor_SMD:C_0603_1608Metric"
-			(at 179.07 86.6648 0)
-			(effects
-				(font
-					(size 1.27 1.27)
-				)
-				(hide yes)
-			)
-		)
-		(property "Datasheet" "~"
-			(at 175.26 87.63 0)
-			(effects
-				(font
-					(size 1.27 1.27)
-				)
-				(hide yes)
-			)
-		)
-		(property "Description" "Unpolarized capacitor"
-			(at 175.26 87.63 0)
-			(effects
-				(font
-					(size 1.27 1.27)
-				)
-				(hide yes)
-			)
-		)
-		(pin "1"
-		)
-		(pin "2"
-		)
-		(instances
-			(project "brainboard"
-				(path "/c4f877e5-ce69-4e50-ab01-826c8aac2c0b/0854ffcf-3a8c-4d5d-b21c-b02dba1777b1"
-					(reference "C48")
-					(unit 1)
-				)
-			)
 		)
 	)
@@
 					(unit 1)
 				)
-			)
-		)
-	)
-	(symbol
-		(lib_id "Device:C")
-		(at 167.64 90.17 90)
-		(unit 1)
-		(exclude_from_sim no)
-		(in_bom yes)
-		(on_board yes)
-		(dnp no)
-		(property "Reference" "C49"
-			(at 166.3699 86.36 0)
-			(effects
-				(font
-					(size 1.27 1.27)
-				)
-				(justify left)
-			)
-		)
-		(property "Value" "1u"
-			(at 168.9099 86.36 0)
-			(effects
-				(font
-					(size 1.27 1.27)
-				)
-				(justify left)
-			)
-		)
-		(property "Footprint" "Capacitor_SMD:C_0603_1608Metric"
-			(at 171.45 89.2048 0)
-			(effects
-				(font
-					(size 1.27 1.27)
-				)
-				(hide yes)
-			)
-		)
-		(property "Datasheet" "~"
-			(at 167.64 90.17 0)
-			(effects
-				(font
-					(size 1.27 1.27)
-				)
-				(hide yes)
-			)
-		)
-		(property "Description" "Unpolarized capacitor"
-			(at 167.64 90.17 0)
-			(effects
-				(font
-					(size 1.27 1.27)
-				)
-				(hide yes)
-			)
-		)
-		(pin "1"
-		)
-		(pin "2"
-		)
-		(instances
-			(project "brainboard"
-				(path "/c4f877e5-ce69-4e50-ab01-826c8aac2c0b/0854ffcf-3a8c-4d5d-b21c-b02dba1777b1"
-					(reference "C49")
-					(unit 1)
-				)
