File: hw/brainboard_carrier/brainboard_carrier.kicad_pcb (KiCad board)
At the start: 2 copper layers, 39 x 109.5 mm, 58 parts, among them J1 3.5mm, J10 3.5mm, J11 Eurorack Brainboard, J12 3.5mm, J2 3.5mm, J3 3.5mm, J4 3.5mm, J5 3.5mm, J6 3.5mm, J7 3.5mm, J8 3.5mm, J9 3.5mm, SW1 SW_Push, SW2 SW_Push, SW3 SW_Push, SW4 SW_Push, U1 TL072

Commit message: Tiny adjustments
Parts:
- removed the G*** at (106.0, 85.9)
- added G***: LOGO, Elemental:elemental-4mm, B.Cu at (136.0, 84.0)
Other:
- board text added: "GND"
- board text added: "Mount module on this side Top facing this direction"
